File: sacre.sch (KiCad schematic (older format))
At the start: 72 parts, among them IC1 ST25DV64KC-IE6S3, J1 USB_B_Micro, J2 Conn_01x24, J3 Con_BATT, M1 Vibration_Motor, Q1 DMP1045U_GSD, Q2 UMH3N, Q3 s8050, Q4 SI1308EDL, SW1 SW, SW2 SW, SW3 SW, SW4 SW, U1 TP4054, U2 ADP2108AUJ-3.3, U3 CP2104, U4 LIS3DH, U5 ESP32-PICO-D4, Y1 RV-8803-C7-TA-QC

Commit message: Clean KiCad project files
Parts:
- IC1: symbol SamacSys_Parts:ST25DV64KC-IE6S3 -> SmartFeedback-rescue:ST25DV64KC-IE6S3-SamacSys_Parts
- S1: footprint SamacSys_Parts:MSK12C02 -> MSK12C02:MSK12C02
Changed lines of the file:
@@
 F 0 "S1" V 2854 6878 50  0000 L CNN
 F 1 "MSK12C02" V 2945 6878 50  0000 L CNN
-F 2 "SamacSys_Parts:MSK12C02" H 3250 6850 50  0001 L CNN
+F 2 "MSK12C02:MSK12C02" H 3250 6850 50  0001 L CNN
 F 3 "https://shouhan.en.made-in-china.com/product/xsMEmqgOAXWB/China-Slide-Switch-Msk12c02-Slide-Switch-on-off-2-Position-1p2t-Spdt-Miniature-Horizontal-SMD-7p-Slide-Switch.html" H 3250 6750 50  0001 L CNN
 F 4 "SMD Toggle Switches" H 3250 6650 50  0001 L CNN "Description"
@@
 $EndComp
 $Comp
-L SamacSys_Parts:ST25DV64KC-IE6S3 IC?
+L SmartFeedback-rescue:ST25DV64KC-IE6S3-SamacSys_Parts IC?
 U 1 1 632E5D21
 P 5700 6950

Commit message: Fix KiCad schematic symbol name
Parts:
- IC1: symbol SmartFeedback-rescue:ST25DV64KC-IE6S3-SamacSys_Parts -> SamacSys_Parts:ST25DV64KC-IE6S3
Changed lines of the file:
@@
 $EndComp
 $Comp
-L SmartFeedback-rescue:ST25DV64KC-IE6S3-SamacSys_Parts IC?
+L SamacSys_Parts:ST25DV64KC-IE6S3 IC?
 U 1 1 632E5D21
 P 5700 6950
