File: power.kicad_sch (KiCad schematic)
At the start: 26 parts, among them J3 USB_C_Receptacle_USB2.0_16P, J4 Con_BATT, Q5 CJ3415, Q6 CJ2312, Q7 UMH3N, SW1 TSC02-TDW1FH3.5, U3 CP2104, U4 ADP2108AUJ-3.3, U5 TP4054

Commit message: se fini
Parts:
- removed J3: USB_C_Receptacle_USB2.0_16P, EasyEDA:USB-C-SMD_TYPE-C-6PIN-2MD-073, symbol Connector:USB_C_Receptacle_USB2.0_16P
- removed J4: Con_BATT, Connector_JST_Custom:JST_PH_S2B-PH-SM4-TB_1x02-1MP_P2.00mm_Horizontal, symbol SmartFeedback-rescue:Conn_01x02-Connector_Generic
- added J3: USB_C_Receptacle_USB2.0_16P, EasyEDA:USB-C-SMD_TYPE-C-16PIN-2MD-073, symbol EasyEDA:USB_C_Receptacle_USB2.0_16P
- added J5: +BATT, Connector_Wire:SolderWirePad_1x01_SMD_3x6mm, symbol Connector:Conn_01x01_Pin
- added J6: -BATT, Connector_Wire:SolderWirePad_1x01_SMD_3x6mm, symbol Connector:Conn_01x01_Pin
- L2: footprint Inductor_SMD:L_0805_2012Metric_Pad1.15x1.40mm_HandSolder -> Inductor_SMD:L_0805_2012Metric
Connections:
- net GND: now also J3.A1B12 (GND), J3.B1A12 (GND), J6.1 (Pin_1)
- net USB_VBUS: now also J3.A4B9 (VBUS), J3.B4A9 (VBUS)
- net VBAT_RAW: now also J5.1 (Pin_1)
- net at C19.1, R15.1: now also J3.13 (SHIELD), J3.14 (GND)
- net USB_D+: now reaches D6.3 (K), U3.3 (D+)
- net USB_D+: now also J3.A6 (D+), J3.B6 (D+)
- net USB_D-: now reaches D6.2 (K), U3.4 (D-)
- net USB_D-: now also J3.A7 (D-), J3.B7 (D-)
- net at R16.1: now also J3.A5 (CC1)
- net at R17.1: now also J3.B5 (CC2)
