File: sacre.kicad_pcb (KiCad board)
At the start: 4 copper layers, 91.4 x 88.4 mm, 77 parts, among them J1 Touch, J2 Screen, J3 USB_C_Receptacle_USB2.0_16P, J5 +BATT, J6 -BATT, M1 Vibration_Motor, Q1 CJ2312, Q2 S8050, Q3 CJ3415, Q4 SI1308EDL, Q5 CJ3415, Q6 CJ2312, Q7 UMH3N, SW1 TSC02-TDW1FH3.5, U1 LIS3DH, U2 ESP32-PICO-D4, U3 CP2104, U4 ADP2108AUJ-3.3, U5 TP4054, Y1 RV-8803-C7-TA-QC

Commit message: Guarda el estado actual del diseño KiCad
Parts:
- J1: footprint Connector_FFC-FPC:Hirose_FH12-6S-0.5SH_1x06-1MP_P0.50mm_Horizontal -> EasyEDA:FPC-SMD_P0.50-6P_QCHF-SM-H2.0
- J2: footprint Connector_FFC:524352471TR250 -> EasyEDA:FPC-SMD_P0.50-24P_QCHF-SM-H2.0
- L1: footprint LQH44PN100MP0L:LQH44PN100MP0L -> Inductor_SMD:L_Vishay_IFSC-1515AH_4x4x1.8mm
- moved R11 1.52 mm to (60.5, 98.0), turned to 180 degrees
- moved J2 1.47 mm to (117.4, 131.9), turned to 180 degrees
- moved J1 0.52 mm to (59.5, 102.1), turned to 180 degrees
- moved L1 0.14 mm to (130.7, 121.7)
Connections:
- J1 pad 1: GND -> SDA
- J1 pad 2: +3V3 -> SCL
- J1 pad 3: Net-(J1-Pin_3) -> INT_TOUCH
- J1 pad 4: INT_TOUCH -> Net-(J1-Pin_4)
- J1 pad 5: SCL -> +3V3
- J1 pad 6: SDA -> GND
- JP1 pad 1: Net-(J1-Pin_3) -> Net-(J1-Pin_4)
- R11 pad 2: Net-(J1-Pin_3) -> Net-(J1-Pin_4)
Routing:
- net Net-(J1-Pin_3): track 33.3 -> 0.00 mm, vias 2 -> 0
- net Net-(J1-Pin_4): track 0.00 -> 32.9 mm, vias 0 -> 2
- net SCL: track 111.5 -> 128.1 mm
- net SDA: track 110.3 -> 121.0 mm
- net INT_TOUCH: track 64.1 -> 67.5 mm
- net PREVGL: track 33.8 -> 32.4 mm
- net +3V3: track 246.6 -> 245.3 mm

Commit message: Corrige SDA y SCL del conector táctil
Connections:
- J1 pad 1: SDA -> SCL
- J1 pad 2: SCL -> SDA
Routing:
- net SDA: track 121.0 -> 121.2 mm, vias 4 -> 6

Commit message: Consolida correcciones eléctricas y documentación
Routing:
- net SCL: track 128.3 -> 118.1 mm
Changed lines of the file:
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@@
-	)
-	(segment
-		(start 58.745 96.655)
-		(end 64.7875 96.655)
-		(width 0.2)
-		(layer "F.Cu")
-		(net "SCL")
 	)
 	(segment
@@
 	)
 	(segment
-		(start 58.24 97.16)
-		(end 58.745 96.655)
-		(width 0.2)
-		(layer "F.Cu")
-		(net "SCL")
-	)
-	(segment
-		(start 66.1 109.4)
+		(start 66.02 109.4)
 		(end 67.5 109.4)
-		(width 0.2)
-		(layer "F.Cu")
-		(net "SCL")
-	)
-	(segment
-		(start 58.23 100.56)
-		(end 58.24 99.3)
 		(width 0.2)
 		(layer "F.Cu")
@@
 		(start 57.88 100.91)
 		(end 57.88 104.02)
-		(width 0.2)
-		(layer "F.Cu")
-		(net "SCL")
-	)
-	(segment
-		(start 58.24 99.3)
-		(end 58.24 97.16)
-		(width 0.2)
-		(layer "F.Cu")
-		(net "SCL")
-	)
-	(segment
-		(start 66.1 109.4)
-		(end 66.02 109.4)
 		(width 0.2)
 		(layer "F.Cu")
@@
 	)
 	(segment
-		(start 68.9 111.6)
-		(end 68.9 111.54)
-		(width 0.2)
-		(layer "In2.Cu")
-		(net "SCL")
-	)
-	(segment
 		(start 78.34 152.8)
 		(end 77.38 152.8)
@@
 	)
 	(segment
-		(start 68.9 111.54)
-		(end 68.84 111.54)
-		(width 0.2)
-		(layer "In2.Cu")
-		(net "SCL")
-	)
-	(segment
 		(start 75.9 151.32)
 		(end 75.42 151.32)
@@
 	)
 	(segment
-		(start 68.84 111.54)
+		(start 68.9 111.6)
 		(end 67.5 110.2)
 		(width 0.2)

Commit message: Sincroniza PCB con esquema: componentes huellas y redes
Parts:
- removed C16, C8: 1uF/50V, Capacitor_SMD:C_0603_1608Metric
- removed C21, C22: 10uF, Capacitor_SMD:C_0603_1608Metric
- removed JP1: Jumper_RES_Touch, Jumper:SolderJumper-2_P1.3mm_Open_TrianglePad1.0x1.5mm
- removed L2: 1uH, Inductor_SMD:L_0805_2012Metric
- removed U4: ADP2108AUJ-3.3, Package_TO_SOT_SMD:TSOT-23-5
- added C23: 1uF, Capacitor_SMD:C_0603_1608Metric, F.Cu at (147.0, 97.0)
- added C24: 4.7uF/25V, Capacitor_SMD:C_0603_1608Metric, F.Cu at (153.0, 97.0)
- added C25: 10uF, Capacitor_SMD:C_0603_1608Metric, F.Cu at (147.0, 85.0)
- added C26: 10uF, Capacitor_SMD:C_0603_1608Metric, F.Cu at (153.0, 85.0)
- added C27: 0.1uF, Capacitor_SMD:C_0603_1608Metric, F.Cu at (159.0, 85.0)
- added C28: 10uF, Capacitor_SMD:C_0603_1608Metric, F.Cu at (159.0, 97.0)
- added C29: 1uF, Capacitor_SMD:C_0603_1608Metric, F.Cu at (165.0, 97.0)
- added C30: 100nF, Capacitor_SMD:C_0603_1608Metric, F.Cu at (165.0, 85.0)
- added C31: 10uF, Capacitor_SMD:C_0603_1608Metric, F.Cu at (171.0, 97.0)
- added C32: 10uF, Capacitor_SMD:C_0603_1608Metric, F.Cu at (147.0, 103.0)
- added D8: MBR0530, Diode_SMD:D_SOD-123, F.Cu at (171.0, 85.0)
- added D9: MBR0530, Diode_SMD:D_SOD-123, F.Cu at (147.0, 91.0)
- added L3: 1uH, Inductor_SMD:L_Changjiang_FTC252012S, F.Cu at (153.0, 103.0)
- added R21: 100K, Resistor_SMD:R_0603_1608Metric, F.Cu at (153.0, 91.0)
- added R22: 10K, Resistor_SMD:R_0603_1608Metric, F.Cu at (159.0, 91.0)
- added R23: 24k, Resistor_SMD:R_0603_1608Metric, F.Cu at (159.0, 103.0)
- added R24: 47k, Resistor_SMD:R_0603_1608Metric, F.Cu at (165.0, 103.0)
- added R25: 100K, Resistor_SMD:R_0603_1608Metric, F.Cu at (165.0, 91.0)
- added R26: 453k, Resistor_SMD:R_0603_1608Metric, F.Cu at (171.0, 103.0)
- added R27: 100k, Resistor_SMD:R_0603_1608Metric, F.Cu at (147.0, 109.0)
- added TP1: RTC_EVI, TestPoint:TestPoint_Pad_D1.0mm, F.Cu at (171.0, 91.0)
- added U6: TLV62568DBVR, Package_TO_SOT_SMD:SOT-23-5, F.Cu at (153.0, 109.0)
- C1, C20: value 1uF -> 0.1uF
- C17: value 0.1uF -> 1uF
- C2: value 10uF -> 0.1uF
- L1: value 10uH/1A -> 47uH; footprint Inductor_SMD:L_Vishay_IFSC-1515AH_4x4x1.8mm -> Inductor_SMD:L_Changjiang_FNR4020S
- R10: value 0.47R -> 2.2R
- R11: value 10K -> 1k
- R19, R7, R8: value 10K -> 5.1k
- R9: value 10K -> 1M0
Connections:
- C1 pad 1: +3V3 -> /VMOTOR
- C20 pad 1: GND -> +3V3
- C20 pad 2: USB_VBUS -> GND
- D1 pad 1: +3V3 -> /VMOTOR
- J1 pad 4: Net-(J1-Pin_4) -> Net-(D8-A)
- J2 pad 21: Net-(J2-Pin_21) -> unconnected-(J2-Pin_21-Pad21)
- J2 pad 6: Net-(J2-Pin_6) -> unconnected-(J2-Pin_6-Pad6)
- M1 pad 1: +3V3 -> /VMOTOR
- Q2 pad 1: GND -> Net-(Q2-B)
- Q2 pad 2: Net-(Q2-B) -> GND
- R11 pad 1: +3V3 -> Net-(D8-A)
- R11 pad 2: Net-(J1-Pin_4) -> RES_TOUCH_CTRL
- U2 pad 10: unconnected-(U2-IO34-Pad10) -> ACC_INT2
- U2 pad 12: GPO -> unconnected-(U2-IO32-Pad12)
- U2 pad 18: ACC_INT2 -> unconnected-(U2-IO12-Pad18)
- U2 pad 21: RTC_EVI -> unconnected-(U2-IO15-Pad21)
- U2 pad 24: unconnected-(U2-IO4-Pad24) -> RES_TOUCH_CTRL
- U2 pad 25: RES_TOUCH -> unconnected-(U2-IO16-Pad25)
- U2 pad 26: unconnected-(U2-VDD_SDIO-Pad26) -> Net-(U2-VDD_SDIO)
- U3 pad 16: unconnected-(U3-VPP-Pad16) -> Net-(U3-VPP)
- U3 pad 5: Net-(U3-VDD) -> +3V3
- U3 pad 6: Net-(U3-VDD) -> +3V3
- U3 pad 7: USB_VBUS -> +3V3
- U3 pad 8: USB_VBUS -> Net-(U3-VBUS)
Routing:
- net unconnected-(U2-IO16-Pad25): track 0.00 -> 28.4 mm, vias 0 -> 2
- net RES_TOUCH: track 28.4 -> 0.00 mm, vias 2 -> 0
- net unconnected-(J2-Pin_6-Pad6): track 0.00 -> 6.55 mm
- net Net-(J2-Pin_6): track 6.55 -> 0.00 mm
- net unconnected-(J2-Pin_21-Pad21): track 0.00 -> 6.22 mm
- net Net-(J2-Pin_21): track 6.22 -> 0.00 mm
- net +3V3: track 245.3 -> 249.0 mm, vias 9 -> 10
- net GND: track 109.5 -> 106.3 mm, vias 83 -> 80
- net Net-(U3-VDD): track 2.15 -> 0.00 mm
- net Net-(Q2-B): track 4.06 -> 5.76 mm, vias 0 -> 2
